File: CAN.kicad_sch (KiCad schematic)
At the start: 4 parts, among them U3 TCAN332G

Commit message: updated to external adc
Parts:
- C10: symbol Device:C -> OpenMC:C; MPN (none) -> CC0603ZRY5V5BB475
- C11: symbol Device:C -> OpenMC:C; MPN (none) -> C1608X5R1H104K080AA
- R22: symbol Device:R_Small_US -> OpenMC:R_Small_US
- U3: value TCAN332G -> TCAN334; symbol Interface_CAN_LIN:TCAN332G -> OpenMC:TCAN332G; MPN (none) -> TCAN334
Other:
- company: Nebula Labs -> (none)
Changed lines of the file:
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@@
 	(title_block
 		(title "CAN Transceiver")
-		(date "2024-04-04")
-		(rev "0.1.1")
-		(company "Nebula Labs")
+		(date "2024-04-07")
+		(rev "0.1")
 		(comment 1 "Author: Orion Serup")
-		(comment 2 "CC BY-SA")
+		(comment 2 "https://github.com/orionserup/OpenMC")
 	)
 	(bus_alias "CAN"
@@
 	)
 	(symbol
-		(lib_id "Device:C")
+		(lib_id "OpenMC:C")
 		(at 106.68 49.53 0)
 		(unit 1)
@@
 			)
 		)
-		(property "MPN" ""
+		(property "MPN" "CC0603ZRY5V5BB475"
 			(at 106.68 49.53 0)
 			(effects
@@
 	)
 	(symbol
-		(lib_id "Device:R_Small_US")
+		(lib_id "OpenMC:R_Small_US")
 		(at 107.95 68.58 0)
 		(unit 1)
@@
 	)
 	(symbol
-		(lib_id "Device:C")
+		(lib_id "OpenMC:C")
 		(at 118.11 49.53 0)
 		(unit 1)
@@
 			)
 		)
-		(property "MPN" ""
+		(property "MPN" "C1608X5R1H104K080AA"
 			(at 118.11 49.53 0)
 			(effects
@@
 	)
 	(symbol
-		(lib_id "Interface_CAN_LIN:TCAN332G")
+		(lib_id "OpenMC:TCAN332G")
 		(at 92.71 68.58 0)
 		(unit 1)
@@
 			)
 		)
-		(property "Value" "TCAN332G"
+		(property "Value" "TCAN334"
 			(at 94.9041 58.42 0)
 			(effects
@@
 			)
 		)
-		(property "MPN" ""
+		(property "MPN" "TCAN334"
 			(at 92.71 68.58 0)
 			(effects
